File: Hardware/PCB/MainBoard.sch (EAGLE design)
At the start: 23 parts, among them IC1 L293D, IC2 L293D, Q1 8MHZ, U1 MCU-ATMEGA32-16PU(DIP40), X1 JST-XH-04-PIN-ROUND-PAD, X2 JST-XH-05-PIN-ROUND-PAD, X3 JST-XH-03-PIN-ROUND-PAD, X4 JST-XH-03-PIN-ROUND-PAD

Commit message: Changes to PCB board
Parts:
- added C7, C8: 12pF, capacitor-wima:C2,5-3
- added JP1: PI, microbuilder:RASBERRYPI_IDC
- added JP2: Right, microbuilder:HEADER-1X13
- added JP3: Left, microbuilder:HEADER-1X13
- added JP4, JP5: (no value), microbuilder:HEADER-1X20ROUND
- added R5: 1k, resistor:R-US_0204/2V
- added R6: 2k, resistor:R-US_0204/2V
- added U$4, U$5, U$6, U$7: MOUNTINGHOLE2.5, microbuilder:MOUNTINGHOLE2.5
- X2: value JST-XH-05-PIN-ROUND-PAD -> (none); device Rembrandt Electronics - JST XH Connectors v1-0:JST-XH-05-PIN-ROUND-PAD -> microbuilder:RASPBERRYPI_B+_IDC
Connections:
- new net 3.3V: JP1.3.3V, JP1.3.3V@1, JP3.1, JP3.9
- new net 5.0V: JP1.5.0V, JP1.5.0V@1, JP2.1, JP2.2
- new net GPIO_HUMIDITY: JP4.4, X2.GPIO_GCLK/GPIO4
- new net GPIO_SERVO: JP5.11, X2.GPIO25/GPIO_GEN6
- new net N$12: JP1.SDA, JP3.2
- new net N$13: JP1.SCL, JP3.3
- new net N$14: JP1.GPIO4, JP3.4
- new net N$15: JP1.GPIO17, JP3.6
- new net N$16: JP1.GPIO21, JP3.7
- new net N$17: JP1.GPIO22_27, JP3.8
- new net N$18: JP1.SPI_MOSI, JP3.10
- new net N$19: JP1.SPI_MISO, JP3.11
- new net N$20: JP1.SPI_SCLK, JP3.12
- new net N$21: JP1.TXD, JP2.4
- new net N$22: JP1.RXD, JP2.5
- new net N$23: JP1.GPIO18, JP2.6
- new net N$24: JP1.GPIO23, JP2.8
- new net N$25: JP1.GPIO24, JP2.9
- new net N$26: JP1.GPIO25, JP2.11
- new net N$27: JP1.#SPI_CE0, JP2.12
- new net N$28: JP1.#SPI_CE1, JP2.13
- new net N$29: JP5.4, X2.GPIO14/TXD0
- new net N$30: JP5.5, X2.GPIO15/RXD0
- new net N$31: JP5.6, X2.GPIO18/GPIO_GEN1
- new net N$32: R5.1
- new net N$33: JP5.9, X2.GPIO24/GPIO_GEN5
- new net N$34: C7.1, C8.1
- new net N$35: JP5.12, X2.GPIO9/SPI_CE0_N
- new net N$36: JP5.13, X2.GPIO7/SPI_CE1_N
- new net N$37: JP5.14, X2.ID_SC/RESERVED
- new net N$38: JP5.16, X2.GPIO12
- new net N$39: JP5.18, X2.GPIO16
- new net N$40: JP5.19, X2.GPIO20
- new net N$41: JP5.20, X2.GPIO21
- new net N$42: JP4.1, X2.3.3V@1
- new net N$43: JP4.2, X2.SDA1/GPIO2
- new net N$44: JP4.3, X2.SCL1/GPIO3
- new net N$46: JP4.6, X2.GPIO_GEN0/GPIO17
- new net N$47: JP4.7, X2.GPIO_GEN2/GPIO27
- new net N$48: JP4.8, X2.GPIO_GEN3/GPIO22
- new net N$49: JP4.9, X2.3.3V@2
- new net N$50: JP4.10, X2.SPI_MOSI/GPIO10
- new net N$51: JP4.11, X2.SPI_MISO/GPIO9
- new net N$52: JP4.12, X2.SPI_SCLK/GPIO11
- new net N$53: JP4.14, X2.RESERVED/ID_SD
- new net N$56: JP4.17, X2.GPIO13
- new net N$57: JP4.18, X2.GPIO19
- new net N$59: JP5.1, X2.5.0V@1
- net GND: now also JP1.GND, JP1.GND@1, JP1.GND@2, JP1.GND@3, JP1.GND@4, JP2.10, JP2.3, JP2.7, JP3.13, JP3.5, JP4.13, JP4.20, JP4.5, JP5.10, JP5.15, JP5.17, JP5.3, JP5.7, R6.2, X2.GND@1, X2.GND@2, X2.GND@3, X2.GND@4, X2.GND@5, X2.GND@6, X2.GND@7, X2.GND@8
- net GPIO_ECHO: now also R5.2, R6.1
- net GPIO_FANS: now also JP4.19, X2.GPIO26; no longer X2-3.S
- net GPIO_LIGHTS: now also JP4.15, X2.GPIO5; no longer X2-1.S
- net GPIO_PUMP: now also JP4.16, X2.GPIO6; no longer X2-2.S
- net GPIO_SOL: no longer X2-5.S
- net GPIO_TRIG: now also JP5.8, X2.GPIO23/GPIO_GEN4
- net N$10: now also C7.2
- net N$11: now also C8.2
- net N$8: now also JP5.2, X2.5.0V@2; no longer X2-4.S
Other:
- note removed: "Raspberry Pi Header"
